Commit message: Change end effector tool frame to have z pointing down, per convension

File: hilgendorf_support/urdf/hilgendorf_macro.xacro (robot description, xacro)
@@ -10,5 +10,5 @@
   <!-- Physical dimensions -->
   <xacro:property name="ur5_mount_angle_offset" value="-0.7853981633974483" />
-  <xacro:property name="robotiq_grip_target_offset" value="0.1" />
+  <xacro:property name="robotiq_grip_target_offset" value="0.125" />
   <xacro:macro name="hilgendorf" params="prefix">
     <!-- Arm mount -->
@@ -45,5 +45,5 @@
       <parent link="${prefix}right_robotiq_85_base_link" />
       <child link="${prefix}right_gripper_target" />
-      <origin xyz="${robotiq_grip_target_offset} 0 0" />
+      <origin xyz="${robotiq_grip_target_offset} 0 0" rpy="0 1.57 0" />
     </joint>
     <link name="${prefix}left_gripper_target" />
@@ -51,5 +51,5 @@
       <parent link="${prefix}left_robotiq_85_base_link" />
       <child link="${prefix}left_gripper_target" />
-      <origin xyz="${robotiq_grip_target_offset} 0 0" />
+      <origin xyz="${robotiq_grip_target_offset} 0 0" rpy="0 1.57 0" />
     </joint>
   </xacro:macro>

Commit message: Disable left arm

File: hilgendorf_support/urdf/hilgendorf_macro.xacro (robot description, xacro)
@@ -16,8 +16,8 @@
     <!-- two UR5 arms -->
     <xacro:ur5_robot prefix="${prefix}right_" joint_limited="true" />
-    <xacro:ur5_robot prefix="${prefix}left_" joint_limited="true" />
+    <!-- <xacro:ur5_robot prefix="${prefix}left_" joint_limited="true" /> -->
     <!-- Grippers -->
     <xacro:robotiq_c2_model prefix="${prefix}right_" />
-    <xacro:robotiq_c2_model prefix="${prefix}left_" />
+    <!-- <xacro:robotiq_c2_model prefix="${prefix}left_" /> -->
     <!-- Connect arms to base -->
     <joint name="${prefix}right_shoulder_to_right_arm" type="fixed">
@@ -26,9 +26,9 @@
       <origin xyz="0.0 0.0 0" rpy="0.0 0.0 ${ur5_mount_angle_offset}" />
     </joint>
-    <joint name="${prefix}left_shoulder_to_left_arm" type="fixed">
-      <parent link="${prefix}left_shoulder" />
-      <child link="${prefix}left_base_link" />
-      <origin xyz="0.0 0.0 0" rpy="0.0 0.0 ${ur5_mount_angle_offset}" />
-    </joint>
+    <!-- <joint name="${prefix}left_shoulder_to_left_arm" type="fixed"> -->
+    <!--   <parent link="${prefix}left_shoulder" /> -->
+    <!--   <child link="${prefix}left_base_link" /> -->
+    <!--   <origin xyz="0.0 0.0 0" rpy="0.0 0.0 ${ur5_mount_angle_offset}" /> -->
+    <!-- </joint> -->
     <!-- Connect gripers to arms -->
     <joint name="${prefix}right_arm_to_eef" type="fixed">
@@ -36,8 +36,8 @@
       <child link="${prefix}right_robotiq_85_adapter_link" />
     </joint>
-    <joint name="${prefix}left_arm_to_eef" type="fixed">
-      <parent link="${prefix}left_ee_link" />
-      <child link="${prefix}left_robotiq_85_adapter_link" />
-    </joint>
+    <!-- <joint name="${prefix}left_arm_to_eef" type="fixed"> -->
+    <!--   <parent link="${prefix}left_ee_link" /> -->
+    <!--   <child link="${prefix}left_robotiq_85_adapter_link" /> -->
+    <!-- </joint> -->
     <!-- Add grip target points for easier path planning -->
     <link name="${prefix}right_gripper_target" />
@@ -47,10 +47,10 @@
       <origin xyz="${robotiq_grip_target_offset} 0 0" rpy="0 1.57 0" />
     </joint>
-    <link name="${prefix}left_gripper_target" />
-    <joint name="${prefix}to_left_gripper_target" type="fixed">
-      <parent link="${prefix}left_robotiq_85_base_link" />
-      <child link="${prefix}left_gripper_target" />
-      <origin xyz="${robotiq_grip_target_offset} 0 0" rpy="0 1.57 0" />
-    </joint>
+    <!-- <link name="${prefix}left_gripper_target" /> -->
+    <!-- <joint name="${prefix}to_left_gripper_target" type="fixed"> -->
+    <!--   <parent link="${prefix}left_robotiq_85_base_link" /> -->
+    <!--   <child link="${prefix}left_gripper_target" /> -->
+    <!--   <origin xyz="${robotiq_grip_target_offset} 0 0" rpy="0 1.57 0" /> -->
+    <!-- </joint> -->
   </xacro:macro>
 </robot>
